File: LDA_Board/LDA_Board.sch (EAGLE design)
At the start: 65 parts, among them IC1 STM32F407ZET, IC3 IS62WV5121655T, K1 B3U-1000P, K2 B3U-1000P, U1 CJT1117-3.3-SOT223, Y1 27.12MHZ

Commit message: 3D打印了盒子
Parts:
- removed BLUETOOTH, USART6: 4p-2.54, Seeed-OPL-Connector:DIP-BLACK-FEMALE-HEADER-VERT(4P-2.54)
- removed C16, C28: 0.5PF 50V, 1-LDA_Board:CAP-(0603)
- removed IC3: IS62WV5121655T, 1-LDA_Board:IS62WV5121655T
- removed K1, K2, RESET: B3U-1000P, 1-LDA_Board:SMD-BUTTON
- removed S1: 5.8X5.8SWITCH, 1-LDA_Board:5.8X5.8SWITCH
- removed SPI2, SPI3: 6p-2.54, Seeed-OPL-Connector:DIP-BLACK-FEMALE-HEADER-VERT(6P-2.54)
- removed SWD: 3p-2.54, 1-LDA_Board:DIP-BLACK-FEMALE-HEADER-VERT(3P-2.54)
- removed U1: CJT1117-3.3-SOT223, 1-LDA_Board:PMIC-CJT1117-3.3(SOT223)
- removed USB1: ST-USB-002A, 1-LDA_Board:MINI-USB-RCPT-B-5PS-R/A-SMD(ST-USB-002A)
- added B-1: SIDE-BUTTON, 1-LDA_Board:SIDE-BUTTON
- added BATTERY-1: BATTERY, 1-LDA_Board:BATTERY
- added D10, D11, D9: BLUE-0402, 1-LDA_Board:LED-(0402)
- added D7: HSMF-C118, 1-LDA_Board:SMD-LED-RGB(4P-1210)
- added HC05-1: BLUETOOTH, 1-LDA_Board:BLUETOOTH
- added MCP73831-1: MCP73831, 1-LDA_Board:MCP73831
- added R14: 2k, 1-LDA_Board:RES-(0402)
- added R15, R16, R17, R25: 10k, 1-LDA_Board:RES-(0402)
- added R18: 20k, 1-LDA_Board:RES-(0402)
- added R19: 0R, 1-LDA_Board:RES-(0402)
- added R20, R21, R22, R23, R24: 510R, 1-LDA_Board:RES-(0402)
- added R26: 1.5k, 1-LDA_Board:RES-(0402)
- added RT9013-1: RT9013, 1-LDA_Board:RT9013
- added SW-1: SWITCH-3P, 1-LDA_Board:SWITCH-3P
- added SW3P-1, SW3P-2: LD-CCB-001, 1-LDA_Board:SWITCH(3P)
- added USB2: ZX62-B-5PA, 1-LDA_Board:MICRO-USB-SMD(ZX62-B-5PA)
- C1, C13, C14, C2, C3: device 1-LDA_Board:CAP-(0603) -> 1-LDA_Board:CAP-(0402)
- C10, C9: value 0.5PF 50V -> 4.7uf; device 1-LDA_Board:CAP-(0603) -> 1-LDA_Board:CAP-(0402)
- C11: value 0.5PF 50V -> 1uf; device 1-LDA_Board:CAP-(0603) -> 1-LDA_Board:CAP-(0402)
- C12: value 0.5PF 50V -> 10uf; device 1-LDA_Board:CAP-(0603) -> 1-LDA_Board:CAP-(0402)
- C15, C17, C18, C19, C20, C21, C22, C23, C24, C25, C26, C27, C8: value 0.5PF 50V -> 104; device 1-LDA_Board:CAP-(0603) -> 1-LDA_Board:CAP-(0402)
- C4: value 104 -> 10uf; device 1-LDA_Board:CAP-(0603) -> 1-LDA_Board:CAP-(0402)
- C5: value 10uf -> 104; device 1-LDA_Board:CAP-(0603) -> 1-LDA_Board:CAP-(0402)
- C6, C7: value 0.5PF 50V -> 22pf; device 1-LDA_Board:CAP-(0603) -> 1-LDA_Board:CAP-(0402)
- D1: value SS14 -> BLUE-0402; device 1-LDA_Board:SS14 -> 1-LDA_Board:LED-(0402)
- D2, D3, D4, D5, D6: value BLUE-0603 -> BLUE-0402; device Seeed-OPL-Diode:SMD-LED-CLEAR-BLUE(0603) -> 1-LDA_Board:LED-(0402)
- D8: value BLUE-0603 -> SS14; device Seeed-OPL-Diode:SMD-LED-CLEAR-BLUE(0603) -> 1-LDA_Board:SS14
- R1, R2: device 1-LDA_Board:RES-(0603) -> 1-LDA_Board:RES-(0402)
- R10, R11, R12, R13, R9: value 1.1M 1/10W -> 510R; device 1-LDA_Board:RES-(0603) -> 1-LDA_Board:RES-(0402)
- R3: value 1.1M 1/10W -> 1M; device 1-LDA_Board:RES-(0603) -> 1-LDA_Board:RES-(0402)
- R4: value 1.1M 1/10W -> 10k; device 1-LDA_Board:RES-(0603) -> 1-LDA_Board:RES-(0402)
- R5, R6, R7: value 10k -> 0R; device 1-LDA_Board:RES-(0603) -> 1-LDA_Board:RES-(0402)
- R8: value 1.1M 1/10W -> 470R; device 1-LDA_Board:RES-(0603) -> 1-LDA_Board:RES-(0402)
- Y1: value 27.12MHZ -> 8MHZ
Connections:
- removed net FSMC_A0: IC1MCU.PF0, IC3SRAM.A0
- removed net FSMC_A1: IC1MCU.PF1, IC3SRAM.A1
- removed net FSMC_A10: IC1MCU.PG0, IC3SRAM.A15
- removed net FSMC_A11: IC1MCU.PG1, IC3SRAM.A16
- removed net FSMC_A12: IC1MCU.PG2, IC3SRAM.A18
- removed net FSMC_A13: IC1MCU.PG3, IC3SRAM.A8
- removed net FSMC_A14: IC1MCU.PG4, IC3SRAM.A9
- removed net FSMC_A15: IC1MCU.PG5, IC3SRAM.A10
- removed net FSMC_A16: IC1MCU.PD11, IC3SRAM.A7
- removed net FSMC_A17: IC1MCU.PD12, IC3SRAM.A6
- removed net FSMC_A18: IC1MCU.PD13, IC3SRAM.A5
- removed net FSMC_A2: IC1MCU.PF2, IC3SRAM.A2
- removed net FSMC_A3: IC1MCU.PF3, IC3SRAM.A3
- removed net FSMC_A4: IC1MCU.PF4, IC3SRAM.A4
- removed net FSMC_A5: IC1MCU.PF5, IC3SRAM.A11
- removed net FSMC_A6: IC1MCU.PF12, IC3SRAM.A17
- removed net FSMC_A7: IC1MCU.PF13, IC3SRAM.A12
- removed net FSMC_A8: IC1MCU.PF14, IC3SRAM.A13
- removed net FSMC_A9: IC1MCU.PF15, IC3SRAM.A14
- removed net FSMC_D0: IC1MCU.PD14, IC3SRAM.I/O0
- removed net FSMC_D1: IC1MCU.PD15, IC3SRAM.I/O1
- removed net FSMC_D10: IC1MCU.PE13, IC3SRAM.I/O10
- removed net FSMC_D11: IC1MCU.PE14, IC3SRAM.I/O11
- removed net FSMC_D12: IC1MCU.PE15, IC3SRAM.I/O12
- removed net FSMC_D13: IC1MCU.PD8, IC3SRAM.I/O13
- removed net FSMC_D14: IC1MCU.PD9, IC3SRAM.I/O14
- removed net FSMC_D15: IC1MCU.PD10, IC3SRAM.I/O15
- removed net FSMC_D2: IC1MCU.PD0, IC3SRAM.I/O2
- removed net FSMC_D3: IC1MCU.PD1, IC3SRAM.I/O3
- removed net FSMC_D4: IC1MCU.PE7, IC3SRAM.I/O4
- removed net FSMC_D5: IC1MCU.PE8, IC3SRAM.I/O5
- removed net FSMC_D6: IC1MCU.PE9, IC3SRAM.I/O6
- removed net FSMC_D7: IC1MCU.PE10, IC3SRAM.I/O7
- removed net FSMC_D8: IC1MCU.PE11, IC3SRAM.I/O8
- removed net FSMC_D9: IC1MCU.PE12, IC3SRAM.I/O9
- removed net FSMC_NBL0: IC1MCU.PE0, IC3SRAM.!LB
- removed net FSMC_NBL1: IC1MCU.PE1, IC3SRAM.!UB
- removed net FSMC_NE3: IC1MCU.PG10, IC3SRAM.!CE, R7.2
- removed net FSMC_NOE: IC1MCU.PD4, IC3SRAM.!OE
- removed net FSMC_NWE: IC1MCU.PD5, IC3SRAM.!WE
- removed net RX6: IC1MCU.PC7, USART6.P$4
- removed net SPI2_CLK: IC1MCU.PB13, SPI2.4
- removed net SPI2_CS: IC1MCU.PB12, SPI2.5
- removed net SPI2_MISO: IC1MCU.PB14, SPI2.3
- removed net SPI2_MOSI: IC1MCU.PB15, SPI2.2
- removed net SPI3_CLK: IC1MCU.PC10, SPI3.4
- removed net SPI3_CS: IC1MCU.PA15, SPI3.5
- removed net SPI3_MISO: IC1MCU.PC11, SPI3.3
- removed net SPI3_MOSI: IC1MCU.PC12, SPI3.2
- removed net TX6: IC1MCU.PC6, USART6.P$3
- new net +3.7V: C12.2, R15.1, RT9013-1.EN, RT9013-1.VIN, SW-1.COM
- new net BATTERY: BATTERY-1.+, C9.2, MCP73831-1.VBAT, SW-1.A
- new net LED6: D9.-, IC1MCU.PC4
- new net LED7: D10.-, IC1MCU.PC5
- new net LED_B: IC1MCU.PG14, R20.1
- new net LED_G: IC1MCU.PG15, R22.1
- new net LED_R: IC1MCU.PG13, R21.1
- new net LI_CHARGE: IC1MCU.PE2, R17.2, R18.1
- new net LI_QUANTITY: IC1MCU.PB0, R15.2, R16.1
- new net N$12: D7.R, R21.2
- new net N$16: D1.-, R8.1
- new net N$17: HC05-1.PIO3, R25.1
- new net N$18: D7.G, R22.2
- new net N$19: HC05-1.PIO1, R26.1
- new net N$20: D11.+, R26.2
- new net N$24: D9.+, R23.2
- new net N$25: D10.+, R24.2
- new net USB_D+: R19.1, USB2.D+
- new net USB_D-: R7.1, USB2.D-
- new net VBUS: D8.A, USB2.VBUS
- net +3V3: now also C11.1, C13.2, C14.2, C15.1, ESP8266.6, HC05-1.VCC, R23.1, R24.1, RT9013-1.VOUT, SW3P-1.A; no longer C11.2, C12.2, C13.1, C14.1, C16.1, C28.2, IC3PWR.VDD@1, IC3PWR.VDD@2, K1.1, R7.1, R8.1, SPI2.6, SPI3.6, U1.OUT, USART6.P$1
- net +5V: now also C10.2, D1.+, D8.C, MCP73831-1.VDD, R17.1; no longer BLUETOOTH.P$1, C15.1, D1.A, ESP8266.6, S1.2.1
- net CLK: now also R7.2; no longer SWD.P$2
- net GBC_LED: now also IC1MCU.PF7; no longer IC1MCU.PC0
- net GND: now also B-1.2, BATTERY-1.-, C1.2, C11.2, C13.1, C14.1, C2.2, C3.2, C6.1, C7.1, C8.1, D11.-, D7.+, HC05-1.CON, HC05-1.GND, MCP73831-1.VSS, R14.2, R16.2, R18.2, R25.2, RT9013-1.GND, SW3P-2.A, USB2.GND, USB2.SHIELD; no longer BLUETOOTH.P$2, C1.1, C11.1, C13.2, C14.2, C16.2, C2.1, C28.1, C3.1, C6.2, C7.2, C8.2, D8.-, IC3PWR.GND@1, IC3PWR.GND@2, K2.1, RESET.2, SPI2.1, SPI3.1, SWD.P$1, U1.GND, USART6.P$2, USB1.GND@1, USB1.GND@2, USB1.GND@3, USB1.GND@4, USB1.GND@5
- net KEY1: now also IC1MCU.PA1, SW3P-2.B; no longer IC1MCU.PE3, K2.2
- net N$10: now also D7.B, R20.2; no longer S1.1.1, USB1.VCC
- net N$11: now also MCP73831-1.PROG, R14.1; no longer D8.+, R8.2
- net N$2: now also C2.1; no longer C3.2
- net N$3: now also C3.1; no longer C2.2
- net N$4: now also IC1MCU.PB2; no longer IC1MCU.PB1
- net N$5: now also C1.1; no longer C1.2
- net N$6: now also MCP73831-1.STAT, R8.2; no longer C10.2, C9.2, D1.C, U1.IN
- net OSC_IN: now also C6.2; no longer C7.1
- net OSC_OUT: now also C7.2; no longer C6.1
- net RESET: now also B-1.1, C8.2; no longer C8.1, RESET.1
- net RX3: now also HC05-1.TXD; no longer BLUETOOTH.P$3
- net SWD: now also R19.2; no longer SWD.P$3
- net TX3: now also HC05-1.RXD; no longer BLUETOOTH.P$4
- net WK_UP: now also SW3P-1.B; no longer K1.2
Other:
- note added: "1、milling需要注意"
- note added: "led顺序交换，程序注意 KEY1引脚改变"
- note removed: "power"
- note removed: "sram"
- note removed: "拓展spi2"
- note removed: "拓展spi3"
- note removed: "拓展usart6"
- moved on the sheet: C1, C10, C11, C12, C13, C14, C17, C18, C19, C2, C20, C21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
