File: LDA_BOX_2/LDA_Board.sch (EAGLE design)
At the start: 77 parts, among them IC1 STM32F407ZET, SW3P-1 LD-CCB-001, SW3P-2 LD-CCB-001, Y1 8MHZ

Commit message: 第二版盒子，器件在一端
Parts:
- removed D1, D10, D9: BLUE-0402, 1-LDA_Board:LED-(0402)
- removed D7: HSMF-C118, 1-LDA_Board:SMD-LED-RGB(4P-1210)
- removed R16, R17: 10k, 1-LDA_Board:RES-(0402)
- removed R18: 20k, 1-LDA_Board:RES-(0402)
- removed R20, R21, R22, R23, R24: 510R, 1-LDA_Board:RES-(0402)
- removed SW3P-1: LD-CCB-001, 1-LDA_Board:SWITCH(3P)
- added LED2-1: DOUBLE_LED, 1-LDA_Board:DOUBLE_LED
- R15: value 10k -> 470R
Connections:
- removed net LED6: D9.-, IC1MCU.PC4
- removed net LED7: D10.-, IC1MCU.PC5
- removed net LED_B: IC1MCU.PG14, R20.1
- removed net LED_G: IC1MCU.PG15, R22.1
- removed net LED_R: IC1MCU.PG13, R21.1
- removed net LI_CHARGE: IC1MCU.PE2, R17.2, R18.1
- removed net LI_QUANTITY: IC1MCU.PB0, R15.2, R16.1
- removed net N$10: D7.B, R20.2
- removed net N$12: D7.R, R21.2
- removed net N$18: D7.G, R22.2
- removed net N$24: D9.+, R23.2
- removed net N$25: D10.+, R24.2
- removed net WK_UP: IC1MCU.PA0, SW3P-1.B
- new net BT_RESET: HC05-1.PIO3, IC1MCU.PE12, R25.1
- net +3.7V: no longer R15.1
- net +3V3: now also R15.1; no longer R23.1, R24.1, SW3P-1.A
- net +5V: now also LED2-1.1; no longer D1.+, R17.1
- net GBC_KEY: now also IC1MCU.PB13; no longer IC1MCU.PF6
- net GBC_LED: now also IC1MCU.PB12; no longer IC1MCU.PF7
- net GND: now also LED2-1.3; no longer D7.+, R16.2, R18.2
- net N$16: now also LED2-1.4; no longer D1.-
- net N$17: now also LED2-1.2, R15.2; no longer HC05-1.PIO3, R25.1
Other:
- note added: "2、flash封装需要修改"
- note added: "3、双色led"
- note removed: "指示模式"
- moved on the sheet: R15, R25
